File: JKW_DIP-VGA-v1.0.sch (EAGLE design)
At the start: 32 parts, among them J1 2X20-CHIP-HEADERS, U1 DS2431P

Commit message: ordered at elecrow
Parts:
- added D6: ES2D, diode:ES2D
- added GND, VIN: WIREPAD3,17/1,3, wirepad:WIREPAD3,17/1,3
- added JP1: (no value), jumper:SJ2W
- added U$5: LOGO_3X3_COPPER, logo:LOGO_3X3_COPPER
- added U$6: LOGO_10X10_SILK, logo:LOGO_10X10_SILK
- added U$9: MP1584EN, power_supply:MP1584EN
- added USB: USBUSB-MICROB-SMT-DIP, Spark:USBUSB-MICROB-SMT-DIP
- R1, R10, R11, R12, R13, R14, R15, R16, R17, R18, R19, R2, R20, R21, R22, R23, R3, R4, R5, R6, R7, R8, R9: device VGA-DIP:RESISTOR -> rcl:R-EU_R0805
Connections:
- new net N$3: JP1.1, USB.VBUS
- new net N$65: D6.A, VIN.P
- new net VCC: J1.ACIN-5V, JP1.2
- new net VIN: D6.C, U$9.VIN
- new net VOUT: JP1.3, U$9.VOUT
- net GND: now also GND.P, U$9.GNDIN, U$9.GNDOUT, USB.GND
Other:
- note added: "Close left = input is already 5V Close right = input is 7 - 28V"
- note added: "Power supply 1"
